File: hardware/power_hv.brd (EAGLE design)
At the start: 75 x 35 mm, 37 parts, among them IC1 MC34063AD, IC2 REG1117, IC3 REG1117, J4 GREEN-2P-5.0, Q1 IRF740

Commit message: set component values; add filter cap on power feedback
Parts:
- added C10: 10n, resistor:C0805
- C2: value (none) -> 220u
- C9: value (none) -> 2.2u
- L1: value (none) -> 220uH
- R1, R2, R3: value 0.33 -> 1
- R5: value 470 -> 750k
- R6: value 3k3 -> 5k6
Connections:
- net GND: now also C10.2
- net N$8: now also C10.1
Routing:
- net N$8: track 20.0 -> 22.0 mm
Changed lines of the file:
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@@
 <drawing>
 <settings>
-<setting alwaysvectorfont="yes"/>
+<setting alwaysvectorfont="no"/>
 <setting verticaltext="up"/>
 </settings>
@@
 <attribute name="VALUE" x="20.955" y="8.89" size="1.27" layer="27" rot="R270"/>
 </element>
-<element name="C2" library="rcl" library_urn="urn:adsk.eagle:library:334" package="140CLH-0810" package3d_urn="urn:adsk.eagle:package:23392/1" value="" x="15.621" y="19.558" smashed="yes">
+<element name="C2" library="rcl" library_urn="urn:adsk.eagle:library:334" package="140CLH-0810" package3d_urn="urn:adsk.eagle:package:23392/1" value="220u" x="15.621" y="19.558" smashed="yes">
 <attribute name="NAME" x="22.306" y="19.358" size="1.27" layer="25" rot="R90"/>
 <attribute name="SPICEPREFIX" value="C" x="15.621" y="19.558" size="1.778" layer="27" display="off"/>
@@
 </element>
 <element name="IC1" library="mc34063" package="SOIC8" value="MC34063AD" x="28.194" y="9.652" rot="R270"/>
-<element name="R1" library="resistor" library_urn="urn:adsk.eagle:library:348" package="R0805" package3d_urn="urn:adsk.eagle:package:26059/1" value="0.33" x="35.433" y="9.398" smashed="yes" rot="R180">
+<element name="R1" library="resistor" library_urn="urn:adsk.eagle:library:348" package="R0805" package3d_urn="urn:adsk.eagle:package:26059/1" value="1" x="35.433" y="9.398" smashed="yes" rot="R180">
 <attribute name="NAME" x="33.528" y="10.033" size="1.27" layer="25" rot="R180"/>
 <attribute name="VALUE" x="34.798" y="16.002" size="1.27" layer="27" rot="R180"/>
 </element>
-<element name="R2" library="resistor" library_urn="urn:adsk.eagle:library:348" package="R0805" package3d_urn="urn:adsk.eagle:package:26059/1" value="0.33" x="35.433" y="11.684" smashed="yes" rot="R180">
+<element name="R2" library="resistor" library_urn="urn:adsk.eagle:library:348" package="R0805" package3d_urn="urn:adsk.eagle:package:26059/1" value="1" x="35.433" y="11.684" smashed="yes" rot="R180">
 <attribute name="NAME" x="33.528" y="12.319" size="1.27" layer="25" rot="R180"/>
 <attribute name="VALUE" x="34.798" y="16.002" size="1.27" layer="27" rot="R180"/>
 </element>
-<element name="R3" library="resistor" library_urn="urn:adsk.eagle:library:348" package="R0805" package3d_urn="urn:adsk.eagle:package:26059/1" value="0.33" x="35.433" y="13.97" smashed="yes" rot="R180">
+<element name="R3" library="resistor" library_urn="urn:adsk.eagle:library:348" package="R0805" package3d_urn="urn:adsk.eagle:package:26059/1" value="1" x="35.433" y="13.97" smashed="yes" rot="R180">
 <attribute name="NAME" x="33.528" y="14.605" size="1.27" layer="25" rot="R180"/>
 <attribute name="VALUE" x="34.798" y="16.002" size="1.27" layer="27" rot="R180"/>
@@
 <element name="T1" library="transistor" library_urn="urn:adsk.eagle:library:402" package="SOT23-BEC" package3d_urn="urn:adsk.eagle:package:29919/2" value="" x="14.986" y="12.065" rot="R90"/>
 <element name="D1" library="diode" library_urn="urn:adsk.eagle:library:210" package="SOD80C" package3d_urn="urn:adsk.eagle:package:43405/2" value="PMLL41SOD80C" x="20.955" y="12.827"/>
-<element name="L1" library="rcl" library_urn="urn:adsk.eagle:library:334" package="POWER-CHOKE_WE-TPC" package3d_urn="urn:adsk.eagle:package:23507/1" value="" x="13.081" y="29.464" smashed="yes" rot="R180">
+<element name="L1" library="rcl" library_urn="urn:adsk.eagle:library:334" package="POWER-CHOKE_WE-TPC" package3d_urn="urn:adsk.eagle:package:23507/1" value="220uH" x="13.081" y="29.464" smashed="yes" rot="R180">
 <attribute name="NAME" x="8.961" y="30.409" size="1.778" layer="25" rot="R180"/>
 <attribute name="SPICEPREFIX" value="L" x="13.081" y="29.464" size="1.778" layer="27" rot="R180" display="off"/>
@@
 <attribute name="VALUE" x="6.02" y="11.395" size="1.016" layer="27"/>
 </element>
-<element name="R5" library="resistor" library_urn="urn:adsk.eagle:library:348" package="R0805" package3d_urn="urn:adsk.eagle:package:26059/1" value="470" x="14.478" y="3.302" smashed="yes" rot="R270">
+<element name="R5" library="resistor" library_urn="urn:adsk.eagle:library:348" package="R0805" package3d_urn="urn:adsk.eagle:package:26059/1" value="750k" x="14.478" y="3.302" smashed="yes" rot="R270">
 <attribute name="NAME" x="15.367" y="3.81" size="1.27" layer="25" rot="R270"/>
 <attribute name="VALUE" x="11.938" y="3.937" size="1.27" layer="27" rot="R270"/>
 </element>
-<element name="R6" library="resistor" library_urn="urn:adsk.eagle:library:348" package="R0805" package3d_urn="urn:adsk.eagle:package:26059/1" value="3k3" x="14.478" y="7.62" smashed="yes" rot="R270">
+<element name="R6" library="resistor" library_urn="urn:adsk.eagle:library:348" package="R0805" package3d_urn="urn:adsk.eagle:package:26059/1" value="5k6" x="14.478" y="7.62" smashed="yes" rot="R270">
 <attribute name="NAME" x="15.367" y="7.366" size="1.27" layer="25" rot="R270"/>
 <attribute name="VALUE" x="12.827" y="8.636" size="1.27" layer="27" rot="R270"/>
@@
 <attribute name="SPICEPREFIX" value="L" x="13.97" y="29.464" size="1.778" layer="27" font="vector" rot="R90" display="off"/>
 </element>
-<element name="C9" library="resistor" library_urn="urn:adsk.eagle:library:348" package="E5-8,5" package3d_urn="urn:adsk.eagle:package:25860/1" value="" x="9.144" y="8.89" rot="R90"/>
+<element name="C9" library="resistor" library_urn="urn:adsk.eagle:library:348" package="E5-8,5" package3d_urn="urn:adsk.eagle:package:25860/1" value="2.2u" x="9.144" y="8.89" rot="R90"/>
 <element name="D4" library="diode" library_urn="urn:adsk.eagle:library:210" package="SOD323-W" package3d_urn="urn:adsk.eagle:package:43418/1" value="BAV21WS" x="7.112" y="27.178" rot="R90"/>
+<element name="C10" library="resistor" library_urn="urn:adsk.eagle:library:348" package="C0805" package3d_urn="urn:adsk.eagle:package:26137/1" value="10n" x="25.4" y="5.842" smashed="yes" rot="R180">
+<attribute name="NAME" x="26.924" y="4.826" size="1.27" layer="25" rot="R180"/>
+<attribute name="VALUE" x="26.67" y="8.382" size="1.27" layer="27" rot="R180"/>
+</element>
 </elements>
 <signals>
@@
 <via x="46.863" y="12.446" extent="1-16" drill="0.6"/>
 <via x="46.863" y="7.366" extent="1-16" drill="0.6"/>
+<contactref element="C10" pad="2"/>
 </signal>
 <signal name="N$5">
@@
 <contactref element="R6" pad="2"/>
 <contactref element="IC1" pad="5"/>
-<wire x1="30.794" y1="7.747" x2="27.619" y2="4.572" width="0.4064" layer="1"/>
-<wire x1="14.478" y1="4.252" x2="14.478" y2="4.572" width="0.4064" layer="1"/>
+<wire x1="30.794" y1="7.747" x2="28.889" y2="5.842" width="0.4064" layer="1"/>
+<wire x1="14.478" y1="4.318" x2="14.478" y2="4.572" width="0.4064" layer="1"/>
 <wire x1="14.478" y1="4.572" x2="14.478" y2="6.67" width="0.4064" layer="1"/>
-<wire x1="27.619" y1="4.572" x2="14.478" y2="4.572" width="0.4064" layer="1"/>
+<wire x1="28.889" y1="5.842" x2="26.67" y2="5.842" width="0.4064" layer="1"/>
+<contactref element="C10" pad="1"/>
+<wire x1="25.654" y1="3.81" x2="14.478" y2="3.81" width="0.4064" layer="1"/>
+<wire x1="30.921" y1="7.62" x2="30.794" y2="7.747" width="0.4064" layer="1"/>
+<wire x1="26.35" y1="5.842" x2="26.35" y2="5.522" width="0.4064" layer="1"/>
+<wire x1="26.35" y1="5.522" x2="26.67" y2="5.842" width="0.4064" layer="1"/>
+<wire x1="14.478" y1="4.252" x2="14.478" y2="4.318" width="0.4064" layer="1"/>
+<wire x1="26.416" y1="4.572" x2="26.35" y2="4.638" width="0.4064" layer="1"/>
+<wire x1="14.478" y1="3.81" x2="14.478" y2="4.318" width="0.4064" layer="1"/>
+<wire x1="25.654" y1="3.81" x2="26.416" y2="4.572" width="0.4064" layer="1"/>
+<wire x1="26.35" y1="5.522" x2="26.35" y2="4.638" width="0.4064" layer="1"/>
 </signal>
 <signal name="N$10">
