File: hardware/power_hv.sch (EAGLE design)
At the start: 37 parts, among them IC1 MC34063AD, IC2 REG1117, IC3 REG1117, J4 GREEN-2P-5.0, Q1 IRF740

Commit message: set component values; add filter cap on power feedback
Parts:
- added C10: 10n, resistor:C-EUC0805
- C2: value (none) -> 220u
- C9: value (none) -> 2.2u
- L1: value (none) -> 220uH
- R1, R2, R3: value 0.33 -> 1
- R5: value 470 -> 750k
- R6: value 3k3 -> 5k6
Connections:
- net GND: now also C10.2
- net N$8: now also C10.1
Other:
- moved on the sheet: L2, R5, R6
